File: Macro-Pad/Macro-Pad.kicad_sch (KiCad schematic)
At the start: 1 part, among them U1 ESP32-S3-WROOM-1

Commit message: v1
Parts:
- added C1: 1.0uF, PCM_SparkFun-Capacitor:C_0402_1005Metric, symbol PCM_SparkFun-Capacitor:1.0uF_0402_16V_10%
- added C2: 22uF, PCM_SparkFun-Capacitor:C_0402_1005Metric, symbol PCM_SparkFun-Capacitor:10uF_0402_6.3V_20%
- added J1: USB_C_Receptacle_USB2.0_14P, Connector_USB:USB_C_Receptacle_HRO_TYPE-C-31-M-12, symbol Connector:USB_C_Receptacle_USB2.0_14P
- added KB-SW1, KB-SW2, KB-SW3, KB-SW4: SW_Push, Button_Switch_Keyboard:SW_Cherry_MX_1.00u_PCB, symbol Switch:SW_Push
- added L1: 2.2uH, PCM_SparkFun-Coil:0806, symbol PCM_SparkFun-Coil:2.2uH_0806_1.2A
- added R1, R2: 5.1k, PCM_SparkFun-Resistor:R_0603_1608Metric, symbol PCM_SparkFun-Resistor:5.1k_0603
- added R3: 10k, PCM_SparkFun-Resistor:R_0603_1608Metric, symbol PCM_SparkFun-Resistor:10k_0603
- added RST1: SW_Push, Button_Switch_SMD:SW_SPST_PTS645Sx43SMTR92, symbol Switch:SW_Push
- added U2: TPS62162DSG, Package_SON:Texas_DSG0008A_WSON-8-1EP_2x2mm_P0.5mm_EP0.9x1.6mm_ThermalVias, symbol Regulator_Switching:TPS62162DSG
Connections:
- net at U1.1 (GND), U1.40 (GND), U1.41 (GND): now also C1.2, C2.1, J1.A1 (GND), J1.A12 (GND), J1.B1 (GND), J1.B12 (GND), J1.SH (SHIELD), KB-SW1.1, KB-SW2.1, KB-SW3.1, KB-SW4.1, R1.2, R2.2, RST1.2
- net at U1.13 (USB_D-): now also J1.A7 (D-), J1.B7 (D-)
- net at U1.14 (USB_D+): now also J1.A6 (D+), J1.B6 (D+)
- net at U1.2 (3V3): now also C2.2, L1.1, R3.2, U2.6 (VOS)
- net at U1.26 (IO45): now also KB-SW4.2
- net at U1.27 (IO0): now also RST1.1
- net at U1.3 (EN): now also C1.1, R3.1
- net at U1.33 (IO40): now also KB-SW1.2
- net at U1.34 (IO41): now also KB-SW2.2
- net at U1.35 (IO42): now also KB-SW3.2
- new net: U2.1 (PGND), U2.4 (AGND), U2.5 (FB)
- new net: J1.A4 (VBUS), J1.A9 (VBUS), J1.B4 (VBUS), J1.B9 (VBUS), U2.2 (VIN), U2.3 (EN)
- new net: L1.2, U2.7 (SW)
- new net: J1.B5 (CC2), R2.1
- new net: J1.A5 (CC1), R1.1
Other:
- moved on the sheet: U1

Commit message: fix outdated pcb wiring
Connections:
- net at KB-SW2.2: now also U1.29 (IO36); no longer U1.34 (IO41)
- net at KB-SW4.2: now also U1.31 (IO38); no longer U1.26 (IO45)
- net at KB-SW1.2: now also U1.28 (IO35); no longer U1.33 (IO40)
- net at U1.30 (IO37): now also KB-SW3.2
- net at U1.35 (IO42): no longer KB-SW3.2
Changed lines of the file:
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@@
-	(wire
-		(pts
-			(xy 111.76 34.29) (xy 111.76 66.04)
-		)
-		(stroke
-			(width 0)
-			(type default)
-		)
-	)
 	(wire
 		(pts
@@
 	(wire
 		(pts
-			(xy 111.76 66.04) (xy 50.8 66.04)
-		)
-		(stroke
-			(width 0)
-			(type default)
-		)
-	)
-	(wire
-		(pts
 			(xy 15.24 27.94) (xy 15.24 34.29)
 		)
@@
 	(wire
 		(pts
+			(xy 50.8 45.72) (xy 73.66 45.72)
+		)
+		(stroke
+			(width 0)
+			(type default)
+		)
+	)
+	(wire
+		(pts
 			(xy 55.88 78.74) (xy 55.88 95.25)
 		)
@@
 	(wire
 		(pts
+			(xy 50.8 50.8) (xy 99.06 50.8)
+		)
+		(stroke
+			(width 0)
+			(type default)
+		)
+	)
+	(wire
+		(pts
 			(xy 76.2 113.03) (xy 78.74 113.03)
 		)
@@
 	(wire
 		(pts
+			(xy 86.36 48.26) (xy 86.36 34.29)
+		)
+		(stroke
+			(width 0)
+			(type default)
+		)
+	)
+	(wire
+		(pts
 			(xy 88.9 24.13) (xy 101.6 24.13)
 		)
@@
 	(wire
 		(pts
-			(xy 99.06 34.29) (xy 99.06 63.5)
-		)
-		(stroke
-			(width 0)
-			(type default)
-		)
-	)
-	(wire
-		(pts
 			(xy 76.2 24.13) (xy 76.2 34.29)
 		)
@@
 	(wire
 		(pts
-			(xy 73.66 34.29) (xy 73.66 58.42)
-		)
-		(stroke
-			(width 0)
-			(type default)
-		)
-	)
-	(wire
-		(pts
 			(xy 15.24 19.05) (xy 15.24 27.94)
 		)
@@
 	(wire
 		(pts
-			(xy 86.36 60.96) (xy 50.8 60.96)
-		)
-		(stroke
-			(width 0)
-			(type default)
-		)
-	)
-	(wire
-		(pts
 			(xy 17.78 33.02) (xy 20.32 33.02)
 		)
@@
 	(wire
 		(pts
+			(xy 50.8 48.26) (xy 86.36 48.26)
+		)
+		(stroke
+			(width 0)
+			(type default)
+		)
+	)
+	(wire
+		(pts
 			(xy 55.88 95.25) (xy 55.88 97.79)
 		)
@@
 	(wire
 		(pts
+			(xy 99.06 50.8) (xy 99.06 34.29)
+		)
+		(stroke
+			(width 0)
+			(type default)
+		)
+	)
+	(wire
+		(pts
 			(xy 66.04 92.71) (xy 48.26 92.71)
 		)
@@
 	(wire
 		(pts
-			(xy 73.66 58.42) (xy 50.8 58.42)
-		)
-		(stroke
-			(width 0)
-			(type default)
-		)
-	)
-	(wire
-		(pts
 			(xy 60.96 40.64) (xy 50.8 40.64)
 		)
@@
 	(wire
 		(pts
-			(xy 99.06 63.5) (xy 50.8 63.5)
+			(xy 111.76 53.34) (xy 111.76 34.29)
 		)
 		(stroke
@@
 	(wire
 		(pts
+			(xy 50.8 53.34) (xy 111.76 53.34)
+		)
+		(stroke
+			(width 0)
+			(type default)
+		)
+	)
+	(wire
+		(pts
+			(xy 73.66 45.72) (xy 73.66 34.29)
+		)
+		(stroke
+			(width 0)
+			(type default)
+		)
+	)
+	(wire
+		(pts
 			(xy 86.36 92.71) (xy 91.44 92.71)
 		)
@@
 		)
 		(stroke
-			(width 0)
-			(type default)
-		)
-	)
-	(wire
-		(pts
-			(xy 86.36 34.29) (xy 86.36 60.96)
-		)
-		(stroke

Commit message: change btn name, move traces
Parts:
- renumbered RST1 to BOOT
Changed lines of the file:
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@@
+	)
+	(junction
+		(at 26.67 12.7)
+		(diameter 0)
+		(color 0 0 0 0)
 	)
 	(junction
@@
 	(wire
 		(pts
+			(xy 26.67 16.51) (xy 26.67 12.7)
+		)
+		(stroke
+			(width 0)
+			(type default)
+		)
+	)
+	(wire
+		(pts
 			(xy 76.2 24.13) (xy 76.2 34.29)
 		)
@@
 	(wire
 		(pts
+			(xy 26.67 12.7) (xy 35.56 12.7)
+		)
+		(stroke
+			(width 0)
+			(type default)
+		)
+	)
+	(wire
+		(pts
 			(xy 60.96 40.64) (xy 50.8 40.64)
 		)
@@
 	(wire
 		(pts
-			(xy 20.32 12.7) (xy 35.56 12.7)
+			(xy 20.32 12.7) (xy 26.67 12.7)
 		)
 		(stroke
@@
 		(dnp no)
 		(fields_autoplaced yes)
-		(property "Reference" "RST1"
+		(property "Reference" "BOOT"
 			(at 27.94 11.43 0)
 			(show_name no)
@@
 			(project "Macro-Pad"
 				(path "/992a88e0-714e-4011-b0b3-d8f6dfe24403"
-					(reference "RST1")
+					(reference "BOOT")
 					(unit 1)
 				)

Commit message: re-format everything to save and optimize space
Parts:
- removed C1: 1.0uF, PCM_SparkFun-Capacitor:C_0402_1005Metric, symbol PCM_SparkFun-Capacitor:1.0uF_0402_16V_10%
- removed L1: 2.2uH, PCM_SparkFun-Coil:0806, symbol PCM_SparkFun-Coil:2.2uH_0806_1.2A
- removed U2: TPS62162DSG, Package_SON:Texas_DSG0008A_WSON-8-1EP_2x2mm_P0.5mm_EP0.9x1.6mm_ThermalVias, symbol Regulator_Switching:TPS62162DSG
- added BUCK1: AMS1117-3.3, Package_TO_SOT_SMD:SOT-223-3_TabPin2, symbol Regulator_Linear:AMS1117-3.3
- added C1: 1.0uF, Capacitor_SMD:C_0805_2012Metric_Pad1.18x1.45mm_HandSolder, symbol Device:C_Small
- added IN_CAP1: 10uF, Capacitor_SMD:C_0805_2012Metric_Pad1.18x1.45mm_HandSolder, symbol Device:C_Small
- BOOT1: renamed from BOOT; footprint Button_Switch_SMD:SW_SPST_PTS645Sx43SMTR92 -> Button_Switch_SMD:SW_Push_SPST_NO_Alps_SKRK
- OUT_CAP1: renamed from C2; footprint PCM_SparkFun-Capacitor:C_0402_1005Metric -> Capacitor_SMD:C_0805_2012Metric_Pad1.18x1.45mm_HandSolder
- R1, R2, R3: footprint PCM_SparkFun-Resistor:R_0603_1608Metric -> Resistor_SMD:R_0805_2012Metric_Pad1.20x1.40mm_HandSolder
- renumbered J1 to USBC1
Connections:
- net at USBC1.A4 (VBUS), USBC1.A9 (VBUS), USBC1.B4 (VBUS)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: now also BUCK1.3 (VI), IN_CAP1.1
- net at OUT_CAP1.2, R3.2, U1.2 (3V3): now also BUCK1.2 (VO)
- net at BOOT1.2, KB-SW1.1, KB-SW2.1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: now also BUCK1.1 (GND), C1.2, IN_CAP1.2
- net at R3.1, U1.3 (EN): now also C1.1
